File: Hardware/Layout/Robotic_Finger_Sensor.sch (EAGLE design)
At the start: 14 parts, among them U1 VCNL4040, U3 MS5637

Commit message: Update to LPS25HB pressure sensor
Parts:
- removed U3: MS5637, MS5637:MS5637
- added U2: LPS25HB, LPS25HB:LPS25HB
- C1: value 2.2uF -> 4.7uF; device SparkFun-Capacitors:2.2UF-0603-10V-20% -> SparkFun-Capacitors:4.7UF0603
Connections:
- removed net SCL: J2.SCL, R1.1, U1.SCL, U3.SCL
- removed net SDA: J2.SDA, R2.1, U1.SDA, U3.SDA
- new net SCL/SCK: J2.SCL, R1.1, U1.SCL, U2.SCL/SCK
- new net SDA/MOSI: J2.SDA, R2.1, U1.SDA, U2.SDA/MOSI
- net 3.3V: now also U2.ADDR/MISO, U2.CS, U2.VCC, U2.VDD_IO; no longer U3.VCC
- net GND: now also U2.GND; no longer U3.GND
Other:
- note added: "7-bit I2C Address: 0x5D"
- note added: "LPS25HB Pressure Sensor"
- note removed: "7-bit I2C Adr: 0x76"
- note removed: "MS5637 Pressure Sensor"
- moved on the sheet: C2
Changed lines of the file:
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@@
 <?xml version="1.0" encoding="utf-8"?>
 <!DOCTYPE eagle SYSTEM "eagle.dtd">
-<eagle version="7.7.0">
+<eagle version="9.0.1">
 <drawing>
 <settings>
 <setting alwaysvectorfont="yes"/>
+<setting keepoldvectorfont="yes"/>
 <setting verticaltext="up"/>
 </settings>
@@
 <layer number="59" name="tCarbon" color="7" fill="1" visible="no" active="no"/>
 <layer number="60" name="bCarbon" color="7" fill="1" visible="no" active="no"/>
+<layer number="88" name="SimResults" color="9" fill="1" visible="yes" active="yes"/>
+<layer number="89" name="SimProbes" color="9" fill="1" visible="yes" active="yes"/>
 <layer number="90" name="Modules" color="5" fill="1" visible="yes" active="yes"/>
 <layer number="91" name="Nets" color="2" fill="1" visible="yes" active="yes"/>
@@
 <layer number="230" name="230bmp" color="7" fill="1" visible="yes" active="yes"/>
 <layer number="231" name="231bmp" color="7" fill="1" visible="yes" active="yes"/>
+<layer number="232" name="Eagle3D_PG2" color="7" fill="1" visible="yes" active="yes"/>
+<layer number="233" name="Eagle3D_PG3" color="7" fill="1" visible="yes" active="yes"/>
 <layer number="248" name="Housing" color="7" fill="1" visible="yes" active="yes"/>
 <layer number="249" name="Edge" color="7" fill="1" visible="yes" active="yes"/>
@@
 <part name="R1" library="SparkFun-Resistors" deviceset="2.2KOHM" device="-0603-1/10W-1%" value="2.2k"/>
 <part name="R2" library="SparkFun-Resistors" deviceset="2.2KOHM" device="-0603-1/10W-1%" value="2.2k"/>
-<part name="C1" library="SparkFun-Capacitors" deviceset="2.2UF" device="-0603-10V-20%" value="2.2uF"/>
+<part name="C1" library="SparkFun-Capacitors" deviceset="4.7UF" device="0603" value="4.7uF"/>
 <part name="FRAME2" library="SparkFun-Aesthetics" deviceset="FRAME-LETTER" device=""/>
 <part name="GND4" library="SparkFun" deviceset="GND" device=""/>
@@
 <part name="SUPPLY6" library="SparkFun-PowerSymbols" deviceset="3.3V" device=""/>
 <part name="J2" library="SparkX" deviceset="I2C_STANDARD" device="JS-1MM"/>
-<part name="U3" library="MS5637" deviceset="MS5637" device=""/>
 <part name="C2" library="SparkFun-Capacitors" deviceset="0.1UF" device="-0603-25V-(+80/-20%)" value="0.1uF"/>
 <part name="SUPPLY4" library="SparkFun-PowerSymbols" deviceset="3.3V" device=""/>
@@
 <part name="FD1" library="SparkFun-Aesthetics" deviceset="FIDUCIAL" device="UFIDUCIAL"/>
 <part name="FD2" library="SparkFun-Aesthetics" deviceset="FIDUCIAL" device="UFIDUCIAL"/>
+<part name="U2" library="LPS25HB" deviceset="LPS25HB" device=""/>
+<part name="SUPPLY10" library="SparkFun-PowerSymbols" deviceset="3.3V" device=""/>
 </parts>
 <sheets>
@@
 <wire x1="124.46" y1="66.04" x2="147.32" y2="66.04" width="0.1524" layer="97" style="longdash"/>
 <wire x1="147.32" y1="66.04" x2="147.32" y2="35.56" width="0.1524" layer="97" style="longdash"/>
-<text x="58.42" y="43.18" size="2.032" layer="97" align="top-left">VCC must be 2.5-3.6V
-</text>
+<text x="58.42" y="43.18" size="2.032" layer="97" rot="MR180" align="top-left">VCC must be 2.5-3.6V </text>
 <wire x1="147.32" y1="66.04" x2="248.92" y2="66.04" width="0.1524" layer="97" style="longdash"/>
 <text x="72.644" y="17.272" size="2.032" layer="97" rot="MR180" align="top-left">I2C Port</text>
 <text x="170.942" y="94.234" size="1.778" layer="97">7-bit I2C Adr: 0x60</text>
-<text x="36.322" y="149.352" size="3.048" layer="97">MS5637 Pressure Sensor</text>
-<text x="49.022" y="101.854" size="1.778" layer="97">7-bit I2C Adr: 0x76</text>
+<text x="27.686" y="161.798" size="3.048" layer="97">LPS25HB Pressure Sensor</text>
+<text x="42.672" y="114.554" size="1.778" layer="97">7-bit I2C Address: 0x5D</text>
 <wire x1="124.46" y1="185.42" x2="124.46" y2="66.04" width="0.1524" layer="97" style="longdash"/>
 </plain>
@@
 <instance part="SUPPLY6" gate="G$1" x="220.98" y="142.24"/>
 <instance part="J2" gate="G$1" x="78.74" y="25.4" rot="MR0"/>
-<instance part="U3" gate="U1" x="71.12" y="124.46"/>
-<instance part="C2" gate="G$1" x="38.1" y="124.46"/>
-<instance part="SUPPLY4" gate="G$1" x="55.88" y="127"/>
-<instance part="GND1" gate="1" x="55.88" y="116.84"/>
-<instance part="SUPPLY7" gate="G$1" x="38.1" y="132.08"/>
-<instance part="GND5" gate="1" x="38.1" y="116.84"/>
+<instance part="C2" gate="G$1" x="30.48" y="129.54"/>
+<instance part="SUPPLY4" gate="G$1" x="43.18" y="139.7"/>
+<instance part="GND1" gate="1" x="43.18" y="121.92"/>
+<instance part="SUPPLY7" gate="G$1" x="30.48" y="137.16"/>
+<instance part="GND5" gate="1" x="30.48" y="121.92"/>
 <instance part="FD1" gate="G$1" x="238.76" y="27.94"/>
 <instance part="FD2" gate="G$1" x="236.22" y="27.94"/>
+<instance part="U2" gate="U1" x="60.96" y="132.08"/>
+<instance part="SUPPLY10" gate="G$1" x="78.74" y="142.24"/>
 </instances>
 <busses>
@@
 </segment>
 <segment>
-<pinref part="U3" gate="U1" pin="GND"/>
 <pinref part="GND1" gate="1" pin="GND"/>
-<wire x1="58.42" y1="121.92" x2="55.88" y2="121.92" width="0.1524" layer="91"/>
-<wire x1="55.88" y1="121.92" x2="55.88" y2="119.38" width="0.1524" layer="91"/>
+<wire x1="45.72" y1="127" x2="43.18" y2="127" width="0.1524" layer="91"/>
+<wire x1="43.18" y1="127" x2="43.18" y2="124.46" width="0.1524" layer="91"/>
+<pinref part="U2" gate="U1" pin="GND"/>
 </segment>
 <segment>
 <pinref part="C2" gate="G$1" pin="2"/>
 <pinref part="GND5" gate="1" pin="GND"/>
-<wire x1="38.1" y1="119.38" x2="38.1" y2="121.92" width="0.1524" layer="91"/>
+<wire x1="30.48" y1="124.46" x2="30.48" y2="127" width="0.1524" layer="91"/>
 </segment>
 </net>
-<net name="SCL" class="0">
+<net name="SCL/SCK" class="0">
 <segment>
 <wire x1="71.12" y1="30.48" x2="66.04" y2="30.48" width="0.1524" layer="91"/>
@@
 </segment>
 <segment>
-<pinref part="U3" gate="U1" pin="SCL"/>
-<wire x1="83.82" y1="121.92" x2="86.36" y2="121.92" width="0.1524" layer="91"/>
-<label x="86.36" y="121.92" size="1.27" layer="95" xref="yes"/>
+<wire x1="76.2" y1="132.08" x2="81.28" y2="132.08" width="0.1524" layer="91"/>
+<label x="81.28" y="132.08" size="1.27" layer="95" xref="yes"/>
+<pinref part="U2" gate="U1" pin="SCL/SCK"/>
 </segment>
 </net>
-<net name="SDA" class="0">
+<net name="SDA/MOSI" class="0">
 <segment>
 <wire x1="71.12" y1="27.94" x2="66.04" y2="27.94" width="0.1524" layer="91"/>
@@
 </segment>
 <segment>
-<pinref part="U3" gate="U1" pin="SDA"/>
-<wire x1="83.82" y1="124.46" x2="86.36" y2="124.46" width="0.1524" layer="91"/>
-<label x="86.36" y="124.46" size="1.27" layer="95" xref="yes"/>
+<wire x1="76.2" y1="134.62" x2="81.28" y2="134.62" width="0.1524" layer="91"/>
+<label x="81.28" y="134.62" size="1.27" layer="95" xref="yes"/>
+<pinref part="U2" gate="U1" pin="SDA/MOSI"/>
 </segment>
 </net>
@@
 </segment>
 <segment>
-<pinref part="U3" gate="U1" pin="VCC"/>
 <pinref part="SUPPLY4" gate="G$1" pin="3.3V"/>
-<wire x1="58.42" y1="124.46" x2="55.88" y2="124.46" width="0.1524" layer="91"/>
-<wire x1="55.88" y1="124.46" x2="55.88" y2="127" width="0.1524" layer="91"/>
+<wire x1="45.72" y1="137.16" x2="43.18" y2="137.16" width="0.1524" layer="91"/>
+<wire x1="43.18" y1="137.16" x2="43.18" y2="139.7" width="0.1524" layer="91"/>
+<pinref part="U2" gate="U1" pin="VCC"/>
+<pinref part="U2" gate="U1" pin="VDD_IO"/>
+<wire x1="45.72" y1="134.62" x2="43.18" y2="134.62" width="0.1524" layer="91"/>
+<wire x1="43.18" y1="134.62" x2="43.18" y2="137.16" width="0.1524" layer="91"/>
+<junction x="43.18" y="137.16"/>
 </segment>
 <segment>
 <pinref part="C2" gate="G$1" pin="1"/>
 <pinref part="SUPPLY7" gate="G$1" pin="3.3V"/>
-<wire x1="38.1" y1="132.08" x2="38.1" y2="129.54" width="0.1524" layer="91"/>
+<wire x1="30.48" y1="137.16" x2="30.48" y2="134.62" width="0.1524" layer="91"/>
+</segment>
+<segment>
+<pinref part="U2" gate="U1" pin="ADDR/MISO"/>
+<wire x1="76.2" y1="129.54" x2="78.74" y2="129.54" width="0.1524" layer="91"/>
+<wire x1="78.74" y1="142.24" x2="78.74" y2="129.54" width="0.1524" layer="91"/>
+<pinref part="SUPPLY10" gate="G$1" pin="3.3V"/>
+<pinref part="U2" gate="U1" pin="CS"/>
+<wire x1="76.2" y1="127" x2="78.74" y2="127" width="0.1524" layer="91"/>
+<wire x1="78.74" y1="129.54" x2="78.74" y2="127" width="0.1524" layer="91"/>
+<junction x="78.74" y="129.54"/>
 </segment>
 </net>
@@
 </schematic>
 </drawing>
-<compatibility>
-<note version="6.3" minversion="6.2.2" severity="warning">
-Since Version 6.2.2 text objects can contain more than one line,
-which will not be processed correctly with this version.
-</note>
-</compatibility>
 </eagle>
